Commit message: make the pipeline actually produce a model end to end
The run that this unblocks: 1920 grasps generated, cleaned and balanced to
252 samples, TSDFs and occupancy built, 2 epochs trained, checkpoint written
and found. Before these fixes it could not get past step 1.

Gripper (the reason every dataset was empty). hand.urdf's finger joints run
q=0 OPEN (0.106m apart) to q=0.056 CLOSED, the opposite of the Panda hand
vgn/simulation.py was written against, so execute_grasp's `move(0.0)` --
meant to close on the object -- flung the gripper wide open, and
check_success then required read() > 0.1 * max_opening_width on a gripper
reading zero. Every attempt was scored a failure: 480/480 negative.
clean_balance_data.py drops len(negatives) - len(positives) rows, so it
then deleted the entire dataset and the pipeline carried on over nothing.
Gripper.move()/read() now convert between opening width and joint space,
reset() opens at q=0, and max_opening_width is the measured 0.106m aperture
rather than 0.056, which was the per-finger travel from the xacro.

Grip force. btsim.Joint.set_position drives the joint with the URDF's
effort, i.e. the xacro's nominal 1N, at which the fingers are pushed back
open by the object's weight the moment the arm lifts. Measured over 240
packed-scene grasps: 1N 0.0% success, 20N 10.4%, 50N 11.7%, 150N 0.8% (at
150N light objects get punched out of the scene). Set to 50N.

Thread oversubscription. numpy, Open3D and scikit-image each size an OpenMP
pool to the whole machine, so under --num-proc N every worker tried to use
every core. A scene that takes 0.12s in one process took 2.85s inside a
4-way pool; construct_dataset over 16 scenes went from not finishing in
4m20s to finishing in 20s once the libraries were pinned to one thread per
worker, which has to happen before numpy is imported.

construct_dataset_parallel.py also moves from apply_async-with-callback to
imap_unordered: results are consumed on the calling thread, so a worker's
exception surfaces and progress no longer depends on the pool's callback
thread. It had been stalling with idle workers and results that never
resolved. size/intrinsic are passed in explicitly rather than read from
globals, which spawn does not carry into a worker.

numpy aliases removed in 1.20 (np.bool, np.int, np.long) still in the
vendored ConvONets utils and the dataset loaders; the image pins numpy
1.26.4, so occupancy generation and training both died on them.

run_pipeline.sh: resume on a per-step marker written only after the step
exits 0, instead of on whether its output directory is non-empty -- a step
that died partway still left its directory populated, so the next run
skipped it and built on a half-written dataset. And find the checkpoint
recursively: train_giga.py saves into a timestamped subdirectory of
--logdir, so the old glob reported no checkpoint after a training run that
had in fact worked.

Co-Authored-By: Claude Opus 5 <noreply@anthropic.com>

File: data/urdfs/frida/hand.urdf (robot description, URDF)
Before this commit: robot frida_gripper, 3 links, 2 joints
Joints:
- joint leftfinger: limit lower=0 upper=0.056 effort=1 velocity=8 -> lower=0 upper=0.056 effort=50 velocity=8
- joint rightfinger: limit lower=0 upper=0.056 effort=1 velocity=8 -> lower=0 upper=0.056 effort=50 velocity=8
