Commit message: frida gripper considerations and increased simulation workspace

File: data/urdfs/frida/hand.urdf (robot description, URDF)
Before this commit: robot frida_gripper, 3 links, 2 joints
Joints:
- joint leftfinger: limit lower=0 upper=0.056 effort=50 velocity=8 -> lower=0 upper=0.056 effort=10 velocity=8
- joint rightfinger: limit lower=0 upper=0.056 effort=50 velocity=8 -> lower=0 upper=0.056 effort=10 velocity=8

File: data/urdfs/frida/train/Bottle.urdf (robot description, URDF)
Before this commit: robot Bottle, 1 links, 0 joints
Links:
- link base_link: mass 0.022936 -> 0.022939
